Commit message: inter arm dist param

File: urdf/dual_denso_robot_macro.xacro (robot description, xacro)
@@ -1,8 +1,9 @@
 <?xml version="1.0"?>
 <robot xmlns:xacro="http://wiki.ros.org/xacro">
+  <!-- Edit the value of right_arm_x to reflect actual distance between both arms in meters -->
   <xacro:macro name="dual_denso_robot" params="
     model
-    sim:=False"
-  >
+    sim:=False
+    right_arm_x:=2.0"> <!-- Edit this value -->
     <xacro:arg name="model" default="vm60b1"/>
     <link name="world"/>
@@ -31,5 +32,5 @@
       <parent link="world"/>
       <child link="right_base_link"/>
-      <origin xyz="2 0 0" rpy="0 0 0"/>
+      <origin xyz="${right_arm_x} 0 0" rpy="0 0 0"/>
     </joint>
     <gazebo>
