Commit message: fixed distance xacro

File: config/distance.xacro (robot description, xacro)
@@ -2,4 +2,5 @@
 <robot xmlns:xacro="http://www.ros.org/wiki/xacro">
   <!-- Distance between the two robot bases -->
-  <xacro:property name="right_arm_x" value="1.5"/>
+  <!-- Left arm base is at the world origin -->
+  <xacro:property name="right_arm_x" value="2.0"/>
 </robot>

File: urdf/dual_denso_robot_macro.xacro (robot description, xacro)
@@ -1,13 +1,14 @@
 <?xml version="1.0"?>
 <robot xmlns:xacro="http://wiki.ros.org/xacro">
-  <!-- Edit the value of right_arm_x to reflect actual distance between both arms in meters -->
   <xacro:macro name="dual_denso_robot" params="
     model
-    sim:=False
-    right_arm_x:=2.0"> <!-- Edit this value -->
+    sim:=False"
+  >
     <xacro:arg name="model" default="vm60b1"/>
     <link name="world"/>
     <!-- Include your single-arm macro -->
     <xacro:include filename="$(find manip_facts_lab)/urdf/denso_robot_macro.xacro" />
+    <!-- Include distance property -->
+    <xacro:include filename="$(find manip_facts_lab)/config/distance.xacro" />
     <!-- Left Arm Instance -->
     <xacro:denso_robot
