Commit message: spawn box in rviz

File: config/lift_box.xacro (robot description, xacro)
@@ -9,5 +9,5 @@
     </inertial>
     <visual>
-      <origin xyz="0 0 0.05" rpy="0 0 0"/>
+      <origin xyz="0 0 ${lift_box_size_z / 2}" rpy="0 0 0"/>
       <geometry>
         <box size="${lift_box_size_x} ${lift_box_size_y} ${lift_box_size_z}"/>
@@ -18,5 +18,5 @@
     </visual>
     <collision>
-      <origin xyz="0 0 0.05" rpy="0 0 0"/>
+      <origin xyz="0 0 ${lift_box_size_z / 2}" rpy="0 0 0"/>
       <geometry>
         <box size="${lift_box_size_x} ${lift_box_size_y} ${lift_box_size_z}"/>

Commit message: lift box v1.0 (not working bc of CollisionObj)

File: config/lift_box.xacro (robot description, xacro)
@@ -3,4 +3,6 @@
   <xacro:include filename="$(find dual_denso_arm_manipulation)/config/scene_config.xacro"/>
   <link name="lift_box">
+    <parent link="world"/>
+    <child link="lift_box"/>
     <inertial>
       <origin xyz="0 0 0" rpy="0 0 0"/>

Commit message: working lift motion (w/o collisions)

File: config/lift_box.xacro (robot description, xacro)
@@ -2,27 +2,42 @@
 <robot xmlns:xacro="http://ros.org/wiki/xacro" name="lift_box">
   <xacro:include filename="$(find dual_denso_arm_manipulation)/config/scene_config.xacro"/>
+  <!-- Parameters (can be in scene_config.xacro too) -->
+  <xacro:property name="m"  value="5.0"/>  <!-- mass [kg] -->
+  <xacro:property name="lx" value="${lift_box_size_x}"/>
+  <xacro:property name="ly" value="${lift_box_size_y}"/>
+  <xacro:property name="lz" value="${lift_box_size_z}"/>
+  <!-- Rigid body (free in the world; initial pose comes from spawner) -->
   <link name="lift_box">
-    <parent link="world"/>
-    <child link="lift_box"/>
+    <!-- Correct inertia for a rectangle: Ixx = 1/12 m (ly^2 + lz^2), etc. -->
     <inertial>
       <origin xyz="0 0 0" rpy="0 0 0"/>
-      <mass value="1.0"/>
-      <inertia ixx="0.001" ixy="0.0" ixz="0.0" iyy="0.001" iyz="0.0" izz="0.001"/>
+      <mass value="${m}"/>
+      <inertia
+        ixx="${(m/12.0) * (ly*ly + lz*lz)}"
+        iyy="${(m/12.0) * (lx*lx + lz*lz)}"
+        izz="${(m/12.0) * (lx*lx + ly*ly)}"
+        ixy="0" ixz="0" iyz="0"/>
     </inertial>
+    <!-- Sit on ground by raising the geometry half height -->
     <visual>
-      <origin xyz="0 0 ${lift_box_size_z / 2}" rpy="0 0 0"/>
-      <geometry>
-        <box size="${lift_box_size_x} ${lift_box_size_y} ${lift_box_size_z}"/>
-      </geometry>
-      <material name="orange">
-        <color rgba="1 0.5 0 1"/>
-      </material>
+      <origin xyz="0 0 ${lz/2.0}" rpy="0 0 0"/>
+      <geometry><box size="${lx} ${ly} ${lz}"/></geometry>
+      <material name="orange"><color rgba="1 0.5 0 1"/></material>
     </visual>
     <collision>
-      <origin xyz="0 0 ${lift_box_size_z / 2}" rpy="0 0 0"/>
-      <geometry>
-        <box size="${lift_box_size_x} ${lift_box_size_y} ${lift_box_size_z}"/>
-      </geometry>
+      <origin xyz="0 0 ${lz/2.0}" rpy="0 0 0"/>
+      <geometry><box size="${lx} ${ly} ${lz}"/></geometry>
     </collision>
   </link>
+  <!-- Gazebo contact/friction parameters -->
+  <gazebo reference="lift_box">
+    <!-- High friction so side-pinching can actually hold -->
+    <mu1>1.5</mu1>
+    <mu2>1.5</mu2>
+    <!-- Contact stiffness/damping; tune if still jittery -->
+    <kp>1e6</kp>
+    <kd>1.0</kd>
+    <max_contacts>50</max_contacts>
+    <min_depth>0.001</min_depth>
+  </gazebo>
 </robot>

File: config/scene_config.xacro (robot description, xacro)
@@ -6,11 +6,11 @@
   <!-- Pose and size of additional objects -->
   <xacro:property name="lift_box_x" value="1.0"/>
-  <xacro:property name="lift_box_y" value="0.0"/>
+  <xacro:property name="lift_box_y" value="-0.4"/>
   <xacro:property name="lift_box_z" value="0.0"/>
   <xacro:property name="lift_box_roll" value="0.0"/>
   <xacro:property name="lift_box_pitch" value="0.0"/>
   <xacro:property name="lift_box_yaw" value="0.0"/>
-  <xacro:property name="lift_box_size_x" value="0.5"/>
-  <xacro:property name="lift_box_size_y" value="0.4"/>
-  <xacro:property name="lift_box_size_z" value="0.4"/>
+  <xacro:property name="lift_box_size_x" value="0.8"/>
+  <xacro:property name="lift_box_size_y" value="1.0"/>
+  <xacro:property name="lift_box_size_z" value="1.6"/>
 </robot>

Commit message: box mass parameter

File: config/lift_box.xacro (robot description, xacro)
@@ -3,5 +3,5 @@
   <xacro:include filename="$(find dual_denso_arm_manipulation)/config/scene_config.xacro"/>
   <!-- Parameters (can be in scene_config.xacro too) -->
-  <xacro:property name="m"  value="5.0"/>  <!-- mass [kg] -->
+  <xacro:property name="m"  value="${lift_box_mass}"/>  <!-- mass [kg] -->
   <xacro:property name="lx" value="${lift_box_size_x}"/>
   <xacro:property name="ly" value="${lift_box_size_y}"/>

File: config/scene_config.xacro (robot description, xacro)
@@ -14,3 +14,4 @@
   <xacro:property name="lift_box_size_y" value="1.0"/>
   <xacro:property name="lift_box_size_z" value="1.6"/>
+  <xacro:property name="lift_box_mass" value="5.0"/>
 </robot>

Commit message: lifting box! (w/o collisions)

File: config/lift_box.xacro (robot description, xacro)
@@ -31,5 +31,5 @@
   </link>
   <!-- Gazebo contact/friction parameters -->
-  <gazebo reference="lift_box">
+  <gazebo reference="lift_box_collision">
     <!-- High friction so side-pinching can actually hold -->
     <mu1>1.5</mu1>

File: config/scene_config.xacro (robot description, xacro)
@@ -13,5 +13,5 @@
   <xacro:property name="lift_box_size_x" value="0.8"/>
   <xacro:property name="lift_box_size_y" value="1.0"/>
-  <xacro:property name="lift_box_size_z" value="1.6"/>
-  <xacro:property name="lift_box_mass" value="5.0"/>
+  <xacro:property name="lift_box_size_z" value="1.0"/>
+  <xacro:property name="lift_box_mass" value="1.0"/>
 </robot>

File: urdf/denso_robot_kinematics.xacro (robot description, xacro)
@@ -1,5 +1,15 @@
 <?xml version='1.0' encoding='UTF-8'?>
 <robot xmlns:xacro="http://www.ros.org/wiki/xacro">
-	<xacro:macro name="denso_robot_arm_kinematics" params="namespace model">
+	<xacro:macro name="denso_robot_arm_kinematics" params="
+		namespace
+		model
+		sim:=false
+		ee_mu1:=1.5
+		ee_mu2:=1.3
+		ee_kp:=500000
+		ee_kd:=50
+		ee_maxVel:=0.05
+		ee_minDepth:=0.002"
+	>
 		<!-- <link name="world"/> -->
 		<!-- <joint name="${namespace}joint_w" type="fixed">
@@ -50,5 +60,5 @@
 			<origin rpy="0.000000 0.000000 0.000000" xyz="0.000000 0.000000 0.280000"/>
 			<axis xyz="-0.000000 -0.000000 1.000000"/>
-			<limit effort="1" lower="-2.96705972839036" upper="2.96705972839036" velocity="3.73064127613788"/>
+			<limit effort="300" lower="-2.96705972839036" upper="2.96705972839036" velocity="3.73064127613788"/>
 			<dynamics damping="0" friction="0"/>
 		</joint>
@@ -77,5 +87,5 @@
 			<origin rpy="0.000000 0.000000 0.000000" xyz="0.108999 -0.181083 0.193078"/>
 			<axis xyz="1.000000 -0.000000 -0.000000"/>
-			<limit effort="1" lower="-1.570796326794897" upper="2.356194490192345" velocity="2.48709418409192"/>
+			<limit effort="250" lower="-1.570796326794897" upper="2.356194490192345" velocity="2.48709418409192"/>
 			<dynamics damping="0" friction="0"/>
 		</joint>
@@ -104,5 +114,5 @@
 			<origin rpy="-1.5708 0.000000 0.000000" xyz="-0.039 0.000000 0.519992"/>
 			<axis xyz="1.000000 -0.000000 -0.000000"/>
-			<limit effort="1" lower="-1.396263401595464" upper="2.932153143350472" velocity="2.71540943019156"/>
+			<limit effort="220" lower="-1.396263401595464" upper="2.932153143350472" velocity="2.71540943019156"/>
 			<dynamics damping="0" friction="0"/>
 		</joint>
@@ -131,5 +141,5 @@
 			<origin rpy="0.000000 0.000000 0.000000" xyz="-0.069999 -0.250997 0.10003"/>
 			<axis xyz="-0.000000 -1.000000 -0.000000"/>
-			<limit effort="1" lower="-3.228859116189509" upper="3.228859116189509" velocity="3.73064127613788"/>
+			<limit effort="160" lower="-3.228859116189509" upper="3.228859116189509" velocity="3.73064127613788"/>
 			<dynamics damping="0" friction="0"/>
 		</joint>
@@ -158,5 +168,5 @@
 			<origin rpy="0.000000 0.000000 0.000000" xyz="0.025 -0.33899 0.000000"/>
 			<axis xyz="1.000000 -0.000000 -0.000000"/>
-			<limit effort="1" lower="-2.0943951023932" upper="2.0943951023932" velocity="2.87060410727889"/>
+			<limit effort="120" lower="-2.0943951023932" upper="2.0943951023932" velocity="2.87060410727889"/>
 			<dynamics damping="0" friction="0"/>
 		</joint>
@@ -168,5 +178,5 @@
 				</geometry>
 			</visual>
-			<collision>
+			<collision name="${namespace}J6_collision">
 				<origin rpy="0 0 0" xyz="0 0 0"/>
 				<geometry>
@@ -180,4 +190,24 @@
 			</inertial>
 		</link>
+		<xacro:if value="${sim}">
+			<gazebo reference="${namespace}J6_collision">
+				<surface>
+				<friction>
+					<ode>
+					<mu>${ee_mu1}</mu>
+					<mu2>${ee_mu2}</mu2>
+					</ode>
+				</friction>
+				<contact>
+					<ode>
+					<kp>${ee_kp}</kp>
+					<kd>${ee_kd}</kd>
+					<max_vel>${ee_maxVel}</max_vel>
+					<min_depth>${ee_minDepth}</min_depth>
+					</ode>
+				</contact>
+				</surface>
+			</gazebo>
+			</xacro:if>
 		<joint name="${namespace}joint_6" type="revolute">
 			<parent link="${namespace}J5"/>
@@ -185,5 +215,5 @@
 			<origin rpy="0.000000 0.000000 0.000000" xyz="-0.025 -0.084 0.000000"/>
 			<axis xyz="0.000000 1.000000 -0.000000"/>
-			<limit effort="1" lower="-6.28318530717959" upper="6.28318530717959" velocity="5.96902604182061"/>
+			<limit effort="80" lower="-6.28318530717959" upper="6.28318530717959" velocity="5.96902604182061"/>
 			<dynamics damping="0" friction="0"/>
 		</joint>

File: urdf/denso_robot_macro.xacro (robot description, xacro)
@@ -62,5 +62,5 @@
     <!-- Placeholder for ros2_control transmission which don't yet exist -->
     <!-- links -  main serial chain -->
-    <xacro:denso_robot_arm_kinematics namespace="${namespace}" model="${model}" />
+    <xacro:denso_robot_arm_kinematics namespace="${namespace}" model="${model}" sim="${sim}"/>
     <!-- <gazebo>
 	    <plugin filename="libgazebo_ros2_control.so" name="gazebo_ros2_control">
