Commit message: utils file

File: config/scene_config.xacro (robot description, xacro)
@@ -11,6 +11,6 @@
   <xacro:property name="lift_box_pitch" value="0.0"/>
   <xacro:property name="lift_box_yaw" value="0.0"/>
-  <xacro:property name="lift_box_size_x" value="0.3"/>
-  <xacro:property name="lift_box_size_y" value="0.2"/>
-  <xacro:property name="lift_box_size_z" value="0.2"/>
+  <xacro:property name="lift_box_size_x" value="0.5"/>
+  <xacro:property name="lift_box_size_y" value="0.4"/>
+  <xacro:property name="lift_box_size_z" value="0.4"/>
 </robot>

Commit message: corrected inter-arm distance

File: config/scene_config.xacro (robot description, xacro)
@@ -3,5 +3,5 @@
   <!-- Distance between the two robot bases -->
   <!-- Left arm base is at the world origin -->
-  <xacro:property name="right_arm_x" value="2.0"/>
+  <xacro:property name="right_arm_x" value="1.67"/>
   <!-- Pose and size of additional objects -->
   <xacro:property name="lift_box_x" value="1.0"/>

Commit message: debugging

File: config/scene_config.xacro (robot description, xacro)
@@ -11,7 +11,7 @@
   <xacro:property name="lift_box_pitch" value="0.0"/>
   <xacro:property name="lift_box_yaw" value="0.0"/>
-  <xacro:property name="lift_box_size_x" value="0.8"/>
-  <xacro:property name="lift_box_size_y" value="1.0"/>
-  <xacro:property name="lift_box_size_z" value="1.0"/>
+  <xacro:property name="lift_box_size_x" value="0.4"/>
+  <xacro:property name="lift_box_size_y" value="0.5"/>
+  <xacro:property name="lift_box_size_z" value="0.5"/>
   <xacro:property name="lift_box_mass" value="1.0"/>
 </robot>

File: urdf/dual_denso_robot_macro.xacro (robot description, xacro)
@@ -3,5 +3,5 @@
   <xacro:macro name="dual_denso_robot" params="
     model
-    sim:=False"
+    sim:=false"
   >
     <xacro:arg name="model" default="vm60b1"/>
@@ -17,5 +17,6 @@
       ip_address="192.168.17.21"
       send_format="288"
-      recv_format="292"/>
+      recv_format="292"
+      sim="${sim}"/>
     <joint name="left_arm_mount" type="fixed">
       <parent link="world"/>
@@ -29,5 +30,6 @@
       ip_address="192.168.17.20"
       send_format="288"
-      recv_format="292"/>
+      recv_format="292"
+      sim="${sim}"/>
     <joint name="right_arm_mount" type="fixed">
       <parent link="world"/>
